File: public/showcase/usb-uart/kicad/usb_uart.kicad_sch (KiCad schematic)
At the start: 40 parts, among them J1 12401610E4#2A, J2 UART1, J3 FLOW1, J4 RS485, U1 CH342F, U2 LDO, U3 THVD1450D

Commit message: NOISSUE - Show the two-layer USB UART board
Replace the revision B showcase (50.5 x 38.4 mm, four layers, J_TERM
and an RS-485 surge network) with the two-layer revision A published
in absmach/synth#103 at 4ab0eb9.

- kicad/, source, placement sidecar and reports from that revision.
- Layer tabs drop to top and bottom; the showcase check accepts 2 or 4
  copper layers.
- Regenerate the layer SVGs, schematic SVG, 3D render, GLB, STEP and OG
  image; drop the schematic sidecar and the revision B brief.
- Rewrite QUALIFICATION.md, the prompt and the page metadata for
  revision A: 41.5 x 32.23 mm, 26 nets, 271 segments, 38 vias,
  507.7 mm, no impedance target on the USB pair, fixed RS-485
  termination and no external TVS on A/B.
Parts:
- removed D8: TVS, Package_TO_SOT_SMD:SOT-23, symbol synth:cdsot23_sm712
- removed J_TERM: TERM, Connector_PinHeader_2.54mm:PinHeader_1x02_P2.54mm_Vertical, symbol Connector_Generic:Conn_01x02
- removed R_A, R_B: 10ohm, Resistor_SMD:R_0603_1608Metric, symbol Device:R_US
- H1, H2, H3, H4: footprint MountingHole:MountingHole_3.2mm_M3 -> MountingHole:MountingHole_2.5mm
- J1: value 12401610E4#2A -> TYPE-C-31-M-12; footprint Connector_USB:USB_C_Receptacle_Amphenol_12401610E4-2A -> Connector_USB:USB_C_Receptacle_HRO_TYPE-C-31-M-12; LCSC (none) -> C165948; MPN 12401610E4#2A -> TYPE-C-31-M-12
Connections:
- net MODEM_IDLE is gone; now on net RXD1_MCU: R8.2, U1.1 (ri0), U1.14 (dsr1_tnow1), U1.16 (dcd1), U1.17 (ri1), U1.22 (dsr0), U1.24 (dcd0)
- net RS485_A_BUS is gone; now on net RS485_A: J4.1 (Pin_1), R_TERM.1
- net GND: now also D4.1 (K), D7.1 (K)
- net TXD0: now also R4.1; no longer D4.1 (K)
- net TXD1: now also R7.1; no longer D7.1 (K)
- net VIO: no longer R4.1, R7.1
- net RXD1: now reaches J2.3 (Pin_3), R5.2
- net CTS1: now reaches J3.3 (Pin_3), R6.2
- net LED_TX1: now reaches D7.2 (A), R7.2
- net RS485_B: now reaches J4.2 (Pin_2)
- net RS485_B: now also R_TERM.2, U3.7 (B)
- net LED_PWR: now reaches D3.2 (A), R3.2
- net LED_TX0: now reaches D4.2 (A), R4.2
- net RS485_A: now reaches U3.6 (A)
Other:
- note added: "D4/D7 red LEDs from TXD0/TXD1."
- note added: "J4: A, B, GND. R_TERM 120 ohm 1% across A/B. UART0 TTL is not broken out."
- note removed: "D4/D7 red LEDs from VIO into TXD0/TXD1: TXD idles high, so they light only while data goes out."
- note removed: "J4: A, B, GND. UART0 TTL is not broken out."
- note removed: "R_A/R_B 10 ohm in series and D8 (SM712 class) on the bus side follow TI's 1 kV surge circuit (SLLSEY3E fig. 37). Not surge-tested; R_A/R_B are generic 0603, TI lists pulse-proof parts."
- note removed: "R_TERM 120 ohm 1% across the bus lines through J_TERM: fit the jumper only at an end of the bus."
- moved on the sheet: C2, C3, C4, C5, C6, C7, D1, D2, D3, D4, D5, D6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

Commit message: NOISSUE - Refresh the showcase to #103 as merged
Copy the board, sidecar, reports and KiCad files from absmach/synth at
de3613e (the merge of #103) and regenerate the GLB, STEP, layer SVGs,
schematic SVG, 3D render and OG image from that board.

- 40.99 x 32.23 mm, 273 segments (213 F.Cu, 60 B.Cu), 43 vias, 515.4 mm.
- KiCad DRC 0 errors and 0 warnings, ERC 0 errors and 1 warning.
- USB pair length, skew and return-path figures, 23 layer-change
  warnings, J1 edge clearance and the TX LED behaviour in the limits.
- Reports name Synth e6455e1, the source_revision in release.json.

Signed-off-by: nyagamunene <stevenyaga2014@gmail.com>
Connections:
- net GND: no longer D4.1 (K), D7.1 (K)
- net RXD1_MCU: no longer R8.2, U1.1 (ri0), U1.14 (dsr1_tnow1), U1.16 (dcd1), U1.17 (ri1), U1.22 (dsr0), U1.24 (dcd0)
- net TXD0: now also D4.1 (K); no longer R4.1
- net TXD1: now also D7.1 (K); no longer R7.1
- net VIO: now also R4.1, R7.1
- new net MODEM_IDLE: R8.2, U1.1 (ri0), U1.14 (dsr1_tnow1), U1.16 (dcd1), U1.17 (ri1), U1.22 (dsr0), U1.24 (dcd0)
Other:
- note added: "D4/D7 red LEDs from VIO, sunk into TXD0/TXD1: dark while the line idles, lit on the low bits."
- note removed: "D4/D7 red LEDs from TXD0/TXD1."
- moved on the sheet: C2, C3, C4, C5, C6, C7, D1, D2, D3, D4, D5, D6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
